Commit message: path fix

File: rtb-data/rtbdata/xacro/ufactory_description/lite6/urdf/lite6.urdf (robot description, URDF)
Before this commit: robot lite6, 9 links, 8 joints
Links:
- link link1: geometry collision mesh filename=ufactory_description/lite6/meshes/collision/link1.stl; visual mesh filename=ufactory_description/lite6/meshes/visual/link1.stl
- link link2: geometry collision mesh filename=ufactory_description/lite6/meshes/collision/link2.stl; visual mesh filename=ufactory_description/lite6/meshes/visual/link2.stl
- link link3: geometry collision mesh filename=ufactory_description/lite6/meshes/collision/link3.stl; visual mesh filename=ufactory_description/lite6/meshes/visual/link3.stl
- link link4: geometry collision mesh filename=ufactory_description/lite6/meshes/collision/link4.stl; visual mesh filename=ufactory_description/lite6/meshes/visual/link4.stl
- link link5: geometry collision mesh filename=ufactory_description/lite6/meshes/collision/link5.stl; visual mesh filename=ufactory_description/lite6/meshes/visual/link5.stl
- link link6: geometry collision mesh filename=ufactory_description/lite6/meshes/collision/link6.stl; visual mesh filename=ufactory_description/lite6/meshes/visual/link6.stl
- link link_base: geometry collision mesh filename=ufactory_description/lite6/meshes/collision/base.stl; visual mesh filename=ufactory_description/lite6/meshes/visual/base.stl
- link link_eef: geometry collision mesh filename=ufactory_description/lite6/meshes/collision/gripper_lite.stl; visual mesh filename=ufactory_description/lite6/meshes/visual/gripper_lite.stl

File: rtb-data/rtbdata/xacro/ufactory_description/lite6/urdf/lite6.urdf.xacro (robot description, xacro)
@@ -36,14 +36,14 @@
           rpy="0 0 0" />
         <geometry>
-          <mesh filename="../meshes/visual/base.stl"/>
-        </geometry>
-        <material name="${prefix}White" />
-      </visual>
-      <collision>
-        <origin
-          xyz="0 0 0"
-          rpy="0 0 0" />
-        <geometry>
-          <mesh filename="../meshes/collision/base.stl"/>
+          <mesh filename="ufactory_description/lite6/meshes/visual/base.stl"/>
+        </geometry>
+        <material name="${prefix}White" />
+      </visual>
+      <collision>
+        <origin
+          xyz="0 0 0"
+          rpy="0 0 0" />
+        <geometry>
+          <mesh filename="ufactory_description/lite6/meshes/collision/base.stl"/>
         </geometry>
       </collision>
@@ -69,14 +69,14 @@
           rpy="0 0 0" />
         <geometry>
-          <mesh filename="../meshes/visual/link1.stl"/>
-        </geometry>
-        <material name="${prefix}White" />
-      </visual>
-      <collision>
-        <origin
-          xyz="0 0 0"
-          rpy="0 0 0" />
-        <geometry>
-          <mesh filename="../meshes/collision/link1.stl"/>
+          <mesh filename="ufactory_description/lite6/meshes/visual/link1.stl"/>
+        </geometry>
+        <material name="${prefix}White" />
+      </visual>
+      <collision>
+        <origin
+          xyz="0 0 0"
+          rpy="0 0 0" />
+        <geometry>
+          <mesh filename="ufactory_description/lite6/meshes/collision/link1.stl"/>
         </geometry>
       </collision>
@@ -119,14 +119,14 @@
           rpy="0 0 0" />
         <geometry>
-           <mesh filename="../meshes/visual/link2.stl"/>
-        </geometry>
-        <material name="${prefix}White" />
-      </visual>
-      <collision>
-        <origin
-          xyz="0 0 0"
-          rpy="0 0 0" />
-        <geometry>
-           <mesh filename="../meshes/collision/link2.stl"/>
+           <mesh filename="ufactory_description/lite6/meshes/visual/link2.stl"/>
+        </geometry>
+        <material name="${prefix}White" />
+      </visual>
+      <collision>
+        <origin
+          xyz="0 0 0"
+          rpy="0 0 0" />
+        <geometry>
+           <mesh filename="ufactory_description/lite6/meshes/collision/link2.stl"/>
         </geometry>
       </collision>
@@ -169,14 +169,14 @@
           rpy="0 0 0" />
         <geometry>
-           <mesh filename="../meshes/visual/link3.stl"/>
-        </geometry>
-        <material name="${prefix}White" />
-      </visual>
-      <collision>
-        <origin
-          xyz="0 0 0"
-          rpy="0 0 0" />
-        <geometry>
-           <mesh filename="../meshes/collision/link3.stl"/>
+           <mesh filename="ufactory_description/lite6/meshes/visual/link3.stl"/>
+        </geometry>
+        <material name="${prefix}White" />
+      </visual>
+      <collision>
+        <origin
+          xyz="0 0 0"
+          rpy="0 0 0" />
+        <geometry>
+           <mesh filename="ufactory_description/lite6/meshes/collision/link3.stl"/>
         </geometry>
       </collision>
@@ -219,14 +219,14 @@
           rpy="0 0 0" />
         <geometry>
-           <mesh filename="../meshes/visual/link4.stl"/>
-        </geometry>
-        <material name="${prefix}White" />
-      </visual>
-      <collision>
-        <origin
-          xyz="0 0 0"
-          rpy="0 0 0" />
-        <geometry>
-           <mesh filename="../meshes/collision/link4.stl"/>
+           <mesh filename="ufactory_description/lite6/meshes/visual/link4.stl"/>
+        </geometry>
+        <material name="${prefix}White" />
+      </visual>
+      <collision>
+        <origin
+          xyz="0 0 0"
+          rpy="0 0 0" />
+        <geometry>
+           <mesh filename="ufactory_description/lite6/meshes/collision/link4.stl"/>
         </geometry>
       </collision>
@@ -269,14 +269,14 @@
           rpy="0 0 0" />
         <geometry>
-           <mesh filename="../meshes/visual/link5.stl"/>
-        </geometry>
-        <material name="${prefix}White" />
-      </visual>
-      <collision>
-        <origin
-          xyz="0 0 0"
-          rpy="0 0 0" />
-        <geometry>
-           <mesh filename="../meshes/collision/link5.stl"/>
+           <mesh filename="ufactory_description/lite6/meshes/visual/link5.stl"/>
+        </geometry>
+        <material name="${prefix}White" />
+      </visual>
+      <collision>
+        <origin
+          xyz="0 0 0"
+          rpy="0 0 0" />
+        <geometry>
+           <mesh filename="ufactory_description/lite6/meshes/collision/link5.stl"/>
         </geometry>
       </collision>
@@ -319,5 +319,5 @@
           rpy="0 0 0" />
         <geometry>
-           <mesh filename="../meshes/visual/link6.stl"/>
+           <mesh filename="ufactory_description/lite6/meshes/visual/link6.stl"/>
         </geometry>
         <material name="${prefix}Silver" />
@@ -328,5 +328,5 @@
           rpy="0 0 0" />
         <geometry>
-           <mesh filename="../meshes/collision/link6.stl"/>
+           <mesh filename="ufactory_description/lite6/meshes/collision/link6.stl"/>
         </geometry>
       </collision>
@@ -369,5 +369,5 @@
           rpy="0 0 0" />
         <geometry>
-          <mesh filename="../meshes/visual/gripper_lite.stl"/>
+          <mesh filename="ufactory_description/lite6/meshes/visual/gripper_lite.stl"/>
         </geometry>
         <material name="Silver" />
@@ -378,5 +378,5 @@
           rpy="0 0 0" />
         <geometry>
-          <mesh filename="../meshes/collision/gripper_lite.stl"/>
+          <mesh filename="ufactory_description/lite6/meshes/collision/gripper_lite.stl"/>
         </geometry>
       </collision>

Commit message: add mycobot_280_pi

File: rtb-data/rtbdata/xacro/ufactory_description/lite6/urdf/lite6.urdf (robot description, URDF)
Before this commit: robot lite6, 9 links, 8 joints
Links:
- link link1: geometry collision mesh filename=ufactory_description/lite6/meshes/collision/link1.glb; visual mesh filename=ufactory_description/lite6/meshes/visual/link1.glb
- link link2: geometry collision mesh filename=ufactory_description/lite6/meshes/collision/link2.glb; visual mesh filename=ufactory_description/lite6/meshes/visual/link2.glb
- link link3: geometry collision mesh filename=ufactory_description/lite6/meshes/collision/link3.glb; visual mesh filename=ufactory_description/lite6/meshes/visual/link3.glb
- link link4: geometry collision mesh filename=ufactory_description/lite6/meshes/collision/link4.glb; visual mesh filename=ufactory_description/lite6/meshes/visual/link4.glb
- link link5: geometry collision mesh filename=ufactory_description/lite6/meshes/collision/link5.glb; visual mesh filename=ufactory_description/lite6/meshes/visual/link5.glb
- link link6: geometry collision mesh filename=ufactory_description/lite6/meshes/collision/link6.glb; visual mesh filename=ufactory_description/lite6/meshes/visual/link6.glb
- link link_base: geometry collision mesh filename=ufactory_description/lite6/meshes/collision/base.glb; visual mesh filename=ufactory_description/lite6/meshes/visual/base.glb
- link link_eef: geometry collision mesh filename=ufactory_description/lite6/meshes/collision/gripper_lite.glb; visual mesh filename=ufactory_description/lite6/meshes/visual/gripper_lite.glb

Commit message: some change

File: rtb-data/rtbdata/xacro/ufactory_description/lite6/urdf/lite6.urdf (robot description, URDF)
Before this commit: robot lite6, 9 links, 8 joints
Links:
- link link1: geometry collision mesh filename=ufactory_description/lite6/meshes/collision/link1.stl; visual mesh filename=ufactory_description/lite6/meshes/visual/link1.stl
- link link2: geometry collision mesh filename=ufactory_description/lite6/meshes/collision/link2.stl; visual mesh filename=ufactory_description/lite6/meshes/visual/link2.stl
- link link3: geometry collision mesh filename=ufactory_description/lite6/meshes/collision/link3.stl; visual mesh filename=ufactory_description/lite6/meshes/visual/link3.stl
- link link4: geometry collision mesh filename=ufactory_description/lite6/meshes/collision/link4.stl; visual mesh filename=ufactory_description/lite6/meshes/visual/link4.stl
- link link5: geometry collision mesh filename=ufactory_description/lite6/meshes/collision/link5.stl; visual mesh filename=ufactory_description/lite6/meshes/visual/link5.stl
- link link6: geometry collision mesh filename=ufactory_description/lite6/meshes/collision/link6.stl; visual mesh filename=ufactory_description/lite6/meshes/visual/link6.stl
- link link_base: geometry collision mesh filename=ufactory_description/lite6/meshes/collision/base.stl; visual mesh filename=ufactory_description/lite6/meshes/visual/base.stl
- link link_eef: geometry collision mesh filename=ufactory_description/lite6/meshes/collision/gripper_lite.stl; visual mesh filename=ufactory_description/lite6/meshes/visual/gripper_lite.stl
