Commit message: collision Add

File: rtb-data/rtbdata/xacro/ufactory_description/lite6/urdf/lite6.urdf.xacro (robot description, xacro)
@@ -1,12 +1,11 @@
 <?xml version="1.0" encoding='utf-8'?>
 <robot xmlns:xacro="http://ros.org/wiki/xacro" name="lite6">
-	<xacro:property name="pi" value="3.14159" />
-	<xacro:macro name="lite6" params="prefix
-		joint1_lower_limit  joint1_upper_limit
-		joint2_lower_limit  joint2_upper_limit
-		joint3_lower_limit  joint3_upper_limit
-		joint4_lower_limit  joint4_upper_limit
-		joint5_lower_limit  joint5_upper_limit
-		joint6_lower_limit  joint6_upper_limit"
+  <xacro:macro name="lite6_urdf" params="prefix
+    joint1_lower_limit:=${-2.0*pi}  joint1_upper_limit:=${2.0*pi}
+    joint2_lower_limit:=${-2.61799}  joint2_upper_limit:=${2.61799}
+    joint3_lower_limit:=${-0.061087}  joint3_upper_limit:=${5.235988}
+    joint4_lower_limit:=${-2.0*pi}  joint4_upper_limit:=${2.0*pi}
+    joint5_lower_limit:=${-2.1642}  joint5_upper_limit:=${2.1642}
+    joint6_lower_limit:=${-2.0*pi}  joint6_upper_limit:=${2.0*pi}"
     >
     <material name="${prefix}White">
@@ -20,5 +19,5 @@
         <origin
           xyz="-0.00829544579053192 3.26357432323433E-05 0.0631194584987089"
-          rpy="0 0 ${pi/2}" />
+          rpy="0 0 0" />
         <mass
           value="1.65393501783165" />
@@ -36,14 +35,14 @@
           rpy="0 0 0" />
         <geometry>
-          <mesh filename="ufactory_description/lite6/meshes/visual/base.stl"/>
-        </geometry>
-        <material name="${prefix}White" />
-      </visual>
-      <collision>
-        <origin
-          xyz="0 0 0"
-          rpy="0 0 0" />
-        <geometry>
-          <mesh filename="ufactory_description/lite6/meshes/collision/base.stl"/>
+          <mesh filename="package://ufactory_description/lite6/meshes/visual/base.glb"/>
+        </geometry>
+        <material name="${prefix}White" />
+      </visual>
+      <collision>
+        <origin
+          xyz="0 0 0"
+          rpy="0 0 0" />
+        <geometry>
+          <mesh filename="package://ufactory_description/lite6/meshes/visual/base.glb"/>
         </geometry>
       </collision>
@@ -69,14 +68,14 @@
           rpy="0 0 0" />
         <geometry>
-          <mesh filename="ufactory_description/lite6/meshes/visual/link1.stl"/>
-        </geometry>
-        <material name="${prefix}White" />
-      </visual>
-      <collision>
-        <origin
-          xyz="0 0 0"
-          rpy="0 0 0" />
-        <geometry>
-          <mesh filename="ufactory_description/lite6/meshes/collision/link1.stl"/>
+          <mesh filename="package://ufactory_description/lite6/meshes/visual/link1.glb"/>
+        </geometry>
+        <material name="${prefix}White" />
+      </visual>
+      <collision>
+        <origin
+          xyz="0 0 0"
+          rpy="0 0 0" />
+        <geometry>
+          <mesh filename="package://ufactory_description/lite6/meshes/visual/link1.glb"/>
         </geometry>
       </collision>
@@ -119,14 +118,14 @@
           rpy="0 0 0" />
         <geometry>
-           <mesh filename="ufactory_description/lite6/meshes/visual/link2.stl"/>
-        </geometry>
-        <material name="${prefix}White" />
-      </visual>
-      <collision>
-        <origin
-          xyz="0 0 0"
-          rpy="0 0 0" />
-        <geometry>
-           <mesh filename="ufactory_description/lite6/meshes/collision/link2.stl"/>
+           <mesh filename="package://ufactory_description/lite6/meshes/visual/link2.glb"/>
+        </geometry>
+        <material name="${prefix}White" />
+      </visual>
+      <collision>
+        <origin
+          xyz="0 0 0"
+          rpy="0 0 0" />
+        <geometry>
+           <mesh filename="package://ufactory_description/lite6/meshes/visual/link2.glb"/>
         </geometry>
       </collision>
@@ -169,14 +168,14 @@
           rpy="0 0 0" />
         <geometry>
-           <mesh filename="ufactory_description/lite6/meshes/visual/link3.stl"/>
-        </geometry>
-        <material name="${prefix}White" />
-      </visual>
-      <collision>
-        <origin
-          xyz="0 0 0"
-          rpy="0 0 0" />
-        <geometry>
-           <mesh filename="ufactory_description/lite6/meshes/collision/link3.stl"/>
+           <mesh filename="package://ufactory_description/lite6/meshes/visual/link3.glb"/>
+        </geometry>
+        <material name="${prefix}White" />
+      </visual>
+      <collision>
+        <origin
+          xyz="0 0 0"
+          rpy="0 0 0" />
+        <geometry>
+           <mesh filename="package://ufactory_description/lite6/meshes/visual/link3.glb"/>
         </geometry>
       </collision>
@@ -219,14 +218,14 @@
           rpy="0 0 0" />
         <geometry>
-           <mesh filename="ufactory_description/lite6/meshes/visual/link4.stl"/>
-        </geometry>
-        <material name="${prefix}White" />
-      </visual>
-      <collision>
-        <origin
-          xyz="0 0 0"
-          rpy="0 0 0" />
-        <geometry>
-           <mesh filename="ufactory_description/lite6/meshes/collision/link4.stl"/>
+           <mesh filename="package://ufactory_description/lite6/meshes/visual/link4.glb"/>
+        </geometry>
+        <material name="${prefix}White" />
+      </visual>
+      <collision>
+        <origin
+          xyz="0 0 0"
+          rpy="0 0 0" />
+        <geometry>
+           <mesh filename="package://ufactory_description/lite6/meshes/visual/link4.glb"/>
         </geometry>
       </collision>
@@ -269,14 +268,14 @@
           rpy="0 0 0" />
         <geometry>
-           <mesh filename="ufactory_description/lite6/meshes/visual/link5.stl"/>
-        </geometry>
-        <material name="${prefix}White" />
-      </visual>
-      <collision>
-        <origin
-          xyz="0 0 0"
-          rpy="0 0 0" />
-        <geometry>
-           <mesh filename="ufactory_description/lite6/meshes/collision/link5.stl"/>
+           <mesh filename="package://ufactory_description/lite6/meshes/visual/link5.glb"/>
+        </geometry>
+        <material name="${prefix}White" />
+      </visual>
+      <collision>
+        <origin
+          xyz="0 0 0"
+          rpy="0 0 0" />
+        <geometry>
+           <mesh filename="package://ufactory_description/lite6/meshes/visual/link5.glb"/>
         </geometry>
       </collision>
@@ -319,5 +318,5 @@
           rpy="0 0 0" />
         <geometry>
-           <mesh filename="ufactory_description/lite6/meshes/visual/link6.stl"/>
+           <mesh filename="package://ufactory_description/lite6/meshes/visual/link6.glb"/>
         </geometry>
         <material name="${prefix}Silver" />
@@ -328,5 +327,5 @@
           rpy="0 0 0" />
         <geometry>
-           <mesh filename="ufactory_description/lite6/meshes/collision/link6.stl"/>
+           <mesh filename="package://ufactory_description/lite6/meshes/visual/link6.glb"/>
         </geometry>
       </collision>
@@ -349,37 +348,5 @@
       <dynamics damping="1.0" friction="1.0"/>
     </joint>
-    <link name="link_eef">
-    <inertial>
-        <origin
-          xyz="0.0 0 0"
-          rpy="0 0 0" />
-        <mass
-          value="0.180" />
-        <inertia
-          ixx="7.726E-05"
-          ixy="1E-06"
-          ixz="4E-07"
-          iyy="8.5665E-05"
-          iyz="-6E-07"
-          izz="1.4814E-04" />
-      </inertial>
-      <visual>
-        <origin
-          xyz="0 0 0"
-          rpy="0 0 0" />
-        <geometry>
-          <mesh filename="ufactory_description/lite6/meshes/visual/gripper_lite.stl"/>
-        </geometry>
-        <material name="Silver" />
-      </visual>
-      <collision>
-        <origin
-          xyz="0 0 0"
-          rpy="0 0 0" />
-        <geometry>
-          <mesh filename="ufactory_description/lite6/meshes/collision/gripper_lite.stl"/>
-        </geometry>
-      </collision>
-    </link>
+    <link name="${prefix}link_eef" />
     <joint
       name="${prefix}joint_eef"
@@ -393,12 +360,5 @@
         link="${prefix}link_eef" />
     </joint>
-    <!-- ROS link_base to ABB World Coordinates transform -->
-    <link name="${prefix}base" />
-    <joint name="${prefix}link_base-base" type="fixed">
-      <origin xyz="0 0 0" rpy="0 0 0"/>
-      <parent link="${prefix}link_base"/>
-      <child link="${prefix}base"/>
-    </joint>
   </xacro:macro>
-  <!--<xacro:lite6_urdf prefix=""/> -->
+  <xacro:lite6_urdf prefix=""/>
 </robot>

File: rtb-data/rtbdata/xacro/ufactory_description/lite6/urdf/lite_gripper_pen.urdf.xacro (robot description, xacro)
@@ -33,5 +33,5 @@
         rpy="0 0 0" />
       <geometry>
-        <mesh filename="package://ufactory_description/lite6/meshes/visual/gripper_lite.glb"/>
+        <mesh filename="package://ufactory_description/lite6/meshes/visual/gripper_lite_pen.glb"/>
       </geometry>
       <material name="White_gripper">
@@ -44,5 +44,5 @@
         rpy="0 0 0" />
       <geometry>
-        <mesh filename="package://ufactory_description/lite6/meshes/collision/gripper_lite.glb"/>
+        <mesh filename="package://ufactory_description/lite6/meshes/collision/gripper_lite_pen.glb"/>
       </geometry>
     </collision>
