Commit message: mycobot fix

File: rtb-data/rtbdata/xacro/elephant_robotics/mycobot_280_pi/urdf/mycobot_280_pi.urdf (robot description, URDF)
Before this commit: robot firefighter, 8 links, 7 joints
Joints:
- joint g_base_to_joint1: axis 0 0 0 -> 0 0 1; type fixed -> revolute

Commit message: mycobot modification

File: rtb-data/rtbdata/xacro/elephant_robotics/mycobot_280_pi/urdf/mycobot_280_pi.urdf (robot description, URDF)
Before this commit: robot firefighter, 8 links, 7 joints
Links:
- removed link g_base
- added link link_eef, mass 1.0; collision mesh filename=cube.obj scale=0.001 0.001 0.001; visual mesh filename=cube.obj scale=0.001 0.001 0.001
Joints:
- removed joint g_base_to_joint1
- added joint joint_eef: type fixed, parent joint6_flange, child link_eef, origin xyz=0 0 0 rpy=0 0 0
